Commit message: 3d changes

File: map-pieces/agent.urdf (robot description, URDF)
Before this commit: robot floor, 1 links, 0 joints
Links:
- link base: mass 0 -> 1; geometry collision box size=.25 .25 1; visual box size=.25 .25 1

File: map-pieces/goal.urdf (robot description, URDF)
Before this commit: robot goal, 1 links, 0 joints
Links:
- link base: mass 0 -> 1

File: map-pieces/unknown.urdf (robot description, URDF)
Before this commit: robot floor, 1 links, 0 joints
Links:
- link base: geometry collision box size=1 1 1; visual box size=.1 .1 .1
